Commit message: update

File: mrl1_description/urdf/mrl1.xacro (robot description, xacro)
@@ -58,5 +58,5 @@
       <mass value="3.6"/>
       <!--inertia ixx="${36*(base_l*base_l+base_h*base_h)/12}" ixy="0.0" ixz="0.0" iyy="${36*(base_w*base_w+base_h*base_h)/12}" iyz="0.0" izz="${36*(base_l*base_l+base_w*base_w)/12}"/-->
-      <inertia ixx="0.2307" ixy="0.0" ixz="0.0" iyy="0.2307" iyz="0.0" izz="0.2307"/>
+      <inertia ixx=".2307" ixy="0.0" ixz="0.0" iyy=".2307" iyz="0.0" izz=".2307"/>
     </inertial>
   </link>
@@ -80,5 +80,5 @@
     <inertial>
       <mass value="0.2"/>
-      <inertia ixx="0.001" ixy="0.0" ixz="0.0" iyy="0.001" iyz="0.0" izz="0.001"/>
+      <inertia ixx=".001" ixy="0.0" ixz="0.0" iyy=".001" iyz="0.0" izz=".001"/>
     </inertial>
   </link>
@@ -108,5 +108,5 @@
     <inertial>
       <mass value="0.2"/>
-      <inertia ixx="0.000001" ixy="0.0" ixz="0.0" iyy="0.000001" iyz="0.0" izz="0.000001"/>
+      <inertia ixx=".001" ixy="0.0" ixz="0.0" iyy=".001" iyz="0.0" izz=".001"/>
     </inertial>
   </link>
@@ -137,5 +137,5 @@
       <mass value="1"/>
       <!--inertia ixx="${0.1*(3*wheel_r^2+wheel_h^2)/12}" ixy="0.0" ixz="0.0" iyy="${0.1*(3*wheel_r^2+wheel_h^2)/12}" iyz="0.0" izz="${0.1*wheel_r^2/2}"/-->
-<inertia ixx="0.0032" ixy="0.0" ixz="0.0" iyy="0.00368" iyz="0.0" izz="0.00368"/>
+<inertia ixx=".0032" ixy="0.0" ixz="0.0" iyy=".00368" iyz="0.0" izz=".00368"/>
     </inertial>
   </link>
@@ -164,5 +164,5 @@
       <mass value="1"/>
       <!--inertia ixx="${0.1*(3*wheel_r^2+wheel_h^2)/12}" ixy="0.0" ixz="0.0" iyy="${0.1*(3*wheel_r^2+wheel_h^2)/12}" iyz="0.0" izz="${0.1*wheel_r^2/2}"/-->
-     <inertia ixx="0.0032" ixy="0.0" ixz="0.0" iyy="0.00368" iyz="0.0" izz="0.00368"/>
+     <inertia ixx=".0032" ixy="0.0" ixz="0.0" iyy=".00368" iyz="0.0" izz=".00368"/>
     </inertial>
   </link>
@@ -266,13 +266,13 @@
         <scan>
           <horizontal>
-            <samples>40</samples>
+            <samples>270</samples>
             <resolution>1</resolution>
-            <min_angle>-1.570796</min_angle>
-            <max_angle>1.570796</max_angle>
+            <min_angle>-2.355</min_angle>
+            <max_angle>2.355</max_angle>
           </horizontal>
         </scan>
         <range>
           <min>0.1</min>
-          <max>3.0</max>
+          <max>2.0</max>
           <resolution>0.01</resolution>
         </range>

File: mrl1_description/urdf/mrl2.xacro (robot description, xacro)
@@ -58,5 +58,5 @@
       <mass value="3.6"/>
       <!--inertia ixx="${36*(base_l*base_l+base_h*base_h)/12}" ixy="0.0" ixz="0.0" iyy="${36*(base_w*base_w+base_h*base_h)/12}" iyz="0.0" izz="${36*(base_l*base_l+base_w*base_w)/12}"/-->
-      <inertia ixx="0.2307" ixy="0.0" ixz="0.0" iyy="0.2307" iyz="0.0" izz="0.2307"/>
+      <inertia ixx=".2307" ixy="0.0" ixz="0.0" iyy=".2307" iyz="0.0" izz=".2307"/>
     </inertial>
   </link>
@@ -80,5 +80,5 @@
     <inertial>
       <mass value="0.2"/>
-      <inertia ixx="0.001" ixy="0.0" ixz="0.0" iyy="0.001" iyz="0.0" izz="0.001"/>
+      <inertia ixx=".001" ixy="0.0" ixz="0.0" iyy=".001" iyz="0.0" izz=".001"/>
     </inertial>
   </link>
@@ -108,5 +108,5 @@
     <inertial>
       <mass value="0.2"/>
-      <inertia ixx="0.000001" ixy="0.0" ixz="0.0" iyy="0.000001" iyz="0.0" izz="0.000001"/>
+      <inertia ixx=".001" ixy="0.0" ixz="0.0" iyy=".001" iyz="0.0" izz=".001"/>
     </inertial>
   </link>
@@ -137,5 +137,5 @@
       <mass value="1"/>
       <!--inertia ixx="${0.1*(3*wheel_r^2+wheel_h^2)/12}" ixy="0.0" ixz="0.0" iyy="${0.1*(3*wheel_r^2+wheel_h^2)/12}" iyz="0.0" izz="${0.1*wheel_r^2/2}"/-->
-<inertia ixx="0.0032" ixy="0.0" ixz="0.0" iyy="0.00368" iyz="0.0" izz="0.00368"/>
+<inertia ixx=".0032" ixy="0.0" ixz="0.0" iyy=".00368" iyz="0.0" izz=".00368"/>
     </inertial>
   </link>
@@ -164,5 +164,5 @@
       <mass value="1"/>
       <!--inertia ixx="${0.1*(3*wheel_r^2+wheel_h^2)/12}" ixy="0.0" ixz="0.0" iyy="${0.1*(3*wheel_r^2+wheel_h^2)/12}" iyz="0.0" izz="${0.1*wheel_r^2/2}"/-->
-     <inertia ixx="0.0032" ixy="0.0" ixz="0.0" iyy="0.00368" iyz="0.0" izz="0.00368"/>
+     <inertia ixx=".0032" ixy="0.0" ixz="0.0" iyy=".00368" iyz="0.0" izz=".00368"/>
     </inertial>
   </link>
@@ -190,5 +190,5 @@
       <mass value="0.1" />
       <origin xyz="0 0 0" rpy="0 0 0"/>
-      <inertia ixx="0.001" ixy="0" ixz="0" iyy="0.001" iyz="0" izz="0.001" />
+      <inertia ixx=".001" ixy="0" ixz="0" iyy=".001" iyz="0" izz=".001" />
     </inertial>
   </link>
@@ -266,13 +266,13 @@
         <scan>
           <horizontal>
-            <samples>40</samples>
+            <samples>270s</samples>
             <resolution>1</resolution>
-            <min_angle>-1.570796</min_angle>
-            <max_angle>1.570796</max_angle>
+            <min_angle>-2.355</min_angle>
+            <max_angle>2.355</max_angle>
           </horizontal>
         </scan>
         <range>
           <min>0.1</min>
-          <max>3.0</max>
+          <max>2.0</max>
           <resolution>0.01</resolution>
         </range>

Commit message: update

File: mrl1_description/urdf/mrl1.xacro (robot description, xacro)
@@ -137,5 +137,5 @@
       <mass value="1"/>
       <!--inertia ixx="${0.1*(3*wheel_r^2+wheel_h^2)/12}" ixy="0.0" ixz="0.0" iyy="${0.1*(3*wheel_r^2+wheel_h^2)/12}" iyz="0.0" izz="${0.1*wheel_r^2/2}"/-->
-<inertia ixx=".0032" ixy="0.0" ixz="0.0" iyy=".00368" iyz="0.0" izz=".00368"/>
+<inertia ixx=".00368" ixy="0.0" ixz="0.0" iyy=".00368" iyz="0.0" izz=".00368"/>
     </inertial>
   </link>
@@ -164,5 +164,5 @@
       <mass value="1"/>
       <!--inertia ixx="${0.1*(3*wheel_r^2+wheel_h^2)/12}" ixy="0.0" ixz="0.0" iyy="${0.1*(3*wheel_r^2+wheel_h^2)/12}" iyz="0.0" izz="${0.1*wheel_r^2/2}"/-->
-     <inertia ixx=".0032" ixy="0.0" ixz="0.0" iyy=".00368" iyz="0.0" izz=".00368"/>
+     <inertia ixx=".00368" ixy="0.0" ixz="0.0" iyy=".00368" iyz="0.0" izz=".00368"/>
     </inertial>
   </link>
@@ -246,14 +246,14 @@
   <gazebo reference="left_wheel">
     <material>Gazebo/black</material>
-    <mu1>0.5</mu1>
-    <mu2>0.5</mu2>
-    <dampingFactor>0.4</dampingFactor>
+    <mu1>132.5</mu1>
+    <mu2>132.5</mu2>
+    <dampingFactor>0.08</dampingFactor>
   </gazebo>
   <!-- Right Wheel -->
   <gazebo reference="right_wheel">
     <material>Gazebo/black</material>
-     <mu1>0.5</mu1>
-     <mu2>0.5</mu2>
-     <dampingFactor>0.4</dampingFactor>
+     <mu1>132.5</mu1>
+     <mu2>132.5</mu2>
+     <dampingFactor>0.08</dampingFactor>
   </gazebo>
   <!-- hokuyo -->
@@ -274,5 +274,5 @@
         <range>
           <min>0.1</min>
-          <max>2.3</max>
+          <max>1.5</max>
           <resolution>0.01</resolution>
         </range>

File: mrl1_description/urdf/mrl2.xacro (robot description, xacro)
@@ -137,5 +137,5 @@
       <mass value="1"/>
       <!--inertia ixx="${0.1*(3*wheel_r^2+wheel_h^2)/12}" ixy="0.0" ixz="0.0" iyy="${0.1*(3*wheel_r^2+wheel_h^2)/12}" iyz="0.0" izz="${0.1*wheel_r^2/2}"/-->
-<inertia ixx=".0032" ixy="0.0" ixz="0.0" iyy=".00368" iyz="0.0" izz=".00368"/>
+<inertia ixx=".00368" ixy="0.0" ixz="0.0" iyy=".00368" iyz="0.0" izz=".00368"/>
     </inertial>
   </link>
@@ -164,5 +164,5 @@
       <mass value="1"/>
       <!--inertia ixx="${0.1*(3*wheel_r^2+wheel_h^2)/12}" ixy="0.0" ixz="0.0" iyy="${0.1*(3*wheel_r^2+wheel_h^2)/12}" iyz="0.0" izz="${0.1*wheel_r^2/2}"/-->
-     <inertia ixx=".0032" ixy="0.0" ixz="0.0" iyy=".00368" iyz="0.0" izz=".00368"/>
+     <inertia ixx=".00368" ixy="0.0" ixz="0.0" iyy=".00368" iyz="0.0" izz=".00368"/>
     </inertial>
   </link>
@@ -246,14 +246,14 @@
   <gazebo reference="left_wheel">
     <material>Gazebo/black</material>
-    <mu1>0.5</mu1>
-    <mu2>0.5</mu2>
-    <dampingFactor>0.4</dampingFactor>
+    <mu1>132.5</mu1>
+    <mu2>132.5</mu2>
+    <dampingFactor>0.08</dampingFactor>
   </gazebo>
   <!-- Right Wheel -->
   <gazebo reference="right_wheel">
     <material>Gazebo/black</material>
-     <mu1>0.5</mu1>
-     <mu2>0.5</mu2>
-     <dampingFactor>0.4</dampingFactor>
+     <mu1>132.5</mu1>
+     <mu2>132.5</mu2>
+     <dampingFactor>0.08</dampingFactor>
   </gazebo>
   <!-- hokuyo -->
@@ -274,5 +274,5 @@
         <range>
           <min>0.1</min>
-          <max>2.0</max>
+          <max>1.5</max>
           <resolution>0.01</resolution>
         </range>
